File: power.sch (KiCad schematic (older format))
At the start: 21 parts

Commit message: Add power supplies
Parts:
- removed C?: 470p, symbol Device:C
- removed C? (x6): 47u, symbol Device:C_Small
- removed D?: SS14F, symbol Device:D_Schottky
- removed R?: 330m 1/2W, symbol Device:R
- removed U?: MC34063AD, Package_SO:SOIC-8_3.9x4.9mm_P1.27mm, symbol Regulator_Switching:MC34063AD
- added C22, C23, C24, C25: 1u, Capacitor_SMD:C_0603_1608Metric_Pad1.05x0.95mm_HandSolder, symbol Device:C_Small
- added NT1: Net-Tie_4, NetTie:NetTie-4_SMD_Pad2.0mm, symbol Device:Net-Tie_4
- added R12: 27k, Resistor_SMD:R_0603_1608Metric_Pad1.05x0.95mm_HandSolder, symbol Device:R
- added R13: 120k, Resistor_SMD:R_0603_1608Metric_Pad1.05x0.95mm_HandSolder, symbol Device:R
- added U6: FM1613, Package_SO:SOIC-8_3.9x4.9mm_P1.27mm, symbol solder-station:FM1613
- added U7, U8: XC6201P332, Package_TO_SOT_SMD:SOT-23-5, symbol solder-station:XC6201P332
- C17, C18, C19, C20, C21: renamed from C?; footprint (none) -> Capacitor_SMD:C_0603_1608Metric_Pad1.05x0.95mm_HandSolder
- JP1: renamed from JP?; footprint (none) -> Resistor_SMD:R_0603_1608Metric_Pad1.05x0.95mm_HandSolder
- L1: renamed from L?; value 3.3u -> 4.7u; footprint (none) -> Inductor_SMD:L_Bourns-SRN4018
- L2: renamed from L?; value 33u -> 4.7u; footprint (none) -> Inductor_SMD:L_Bourns-SRN4018
- R14: renamed from R?; value R -> 475k; footprint (none) -> Resistor_SMD:R_0603_1608Metric_Pad1.05x0.95mm_HandSolder
- R15: renamed from R?; value R -> 150k; footprint (none) -> Resistor_SMD:R_0603_1608Metric_Pad1.05x0.95mm_HandSolder
- R16: renamed from R?; value 330m 1/2W -> 150m; footprint (none) -> Resistor_SMD:R_0603_1608Metric_Pad1.05x0.95mm_HandSolder
Connections:
- net labels added: +24V, +3.3V, +3.3VA, GNDA, GNDD, VCC, VSS
- net labels removed: +12V, GNDPWR
- wire segments 37 -> 46
Other:
- note added: "MAX 1.125A"
- note added: "Star ground"
- note added: "The resistor, inductor, and caps form a filter.\nIn simulation, this means 0.2mV pk-pk ripple"
- note added: "VCC for 74-series logic"
- note added: "~~180kHz"
- note removed: "The resistor, inductor, and caps form a filter.\nIn simulation, this leads to an absurdly clean\npower rail: 6.6e-5V pk-pk @ 100kHz"
- moved on the sheet: C17, C18, C19, C20, C21, JP1, L1, L2, R14, R15, R16

Commit message: Move some things around
Parts:
- added J5: Power, TerminalBlock_MetzConnect:TerminalBlock_MetzConnect_Type011_RT05502HBWC_1x02_P5.00mm_Horizontal, symbol Connector:Conn_01x02_Female
- NT1: value Net-Tie_4 -> Star Ground
Connections:
- net labels removed: VCC, VSS
Other:
- note removed: "VCC for 74-series logic"

Commit message: Fix DRC issues
Connections:
- no-connect marks 0 -> 1
Changed lines of the file:
@@
 L power:+5V #PWR038
 U 1 1 5C59B946
-P 900 2700
-F 0 "#PWR038" H 900 2550 50  0001 C CNN
-F 1 "+5V" V 915 2828 50  0000 L CNN
-F 2 "" H 900 2700 50  0001 C CNN
-F 3 "" H 900 2700 50  0001 C CNN
-	1    900  2700
+P 850 2700
+F 0 "#PWR038" H 850 2550 50  0001 C CNN
+F 1 "+5V" V 865 2828 50  0000 L CNN
+F 2 "" H 850 2700 50  0001 C CNN
+F 3 "" H 850 2700 50  0001 C CNN
+	1    850  2700
 	0    -1   -1   0
 $EndComp
@@
 L power:+5V #PWR040
 U 1 1 5C59F991
-P 900 3950
-F 0 "#PWR040" H 900 3800 50  0001 C CNN
-F 1 "+5V" V 915 4078 50  0000 L CNN
-F 2 "" H 900 3950 50  0001 C CNN
-F 3 "" H 900 3950 50  0001 C CNN
-	1    900  3950
+P 850 3950
+F 0 "#PWR040" H 850 3800 50  0001 C CNN
+F 1 "+5V" V 865 4078 50  0000 L CNN
+F 2 "" H 850 3950 50  0001 C CNN
+F 3 "" H 850 3950 50  0001 C CNN
+	1    850  3950
 	0    -1   -1   0
 $EndComp
@@
 	1    0    0    -1
 $EndComp
+NoConn ~ 950  5250
+$Comp
+L power:+24V #PWR0124
+U 1 1 5C6508E9
+P 2750 5100
+F 0 "#PWR0124" H 2750 4950 50  0001 C CNN
+F 1 "+24V" H 2765 5273 50  0000 C CNN
+F 2 "" H 2750 5100 50  0001 C CNN
+F 3 "" H 2750 5100 50  0001 C CNN
+	1    2750 5100
+	-1   0    0    1
+$EndComp
+$Comp
+L power:GND #PWR0130
+U 1 1 5C6509B8
+P 3200 5100
+F 0 "#PWR0130" H 3200 4850 50  0001 C CNN
+F 1 "GND" H 3205 4927 50  0000 C CNN
+F 2 "" H 3200 5100 50  0001 C CNN
+F 3 "" H 3200 5100 50  0001 C CNN
+	1    3200 5100
+	1    0    0    -1
+$EndComp
+$Comp
+L power:PWR_FLAG #FLG0104
+U 1 1 5C6521C7
+P 2750 5100
+F 0 "#FLG0104" H 2750 5175 50  0001 C CNN
+F 1 "PWR_FLAG" H 2750 5274 50  0000 C CNN
+F 2 "" H 2750 5100 50  0001 C CNN
+F 3 "~" H 2750 5100 50  0001 C CNN
+	1    2750 5100
+	1    0    0    -1
+$EndComp
+$Comp
+L power:PWR_FLAG #FLG0105
+U 1 1 5C652CCD
+P 3200 5100
+F 0 "#FLG0105" H 3200 5175 50  0001 C CNN
+F 1 "PWR_FLAG" H 3200 5274 50  0000 C CNN
+F 2 "" H 3200 5100 50  0001 C CNN
+F 3 "~" H 3200 5100 50  0001 C CNN
+	1    3200 5100
+	1    0    0    -1
+$EndComp
+$Comp
+L power:PWR_FLAG #FLG0107
+U 1 1 5C6542D9
+P 3200 5600
+F 0 "#FLG0107" H 3200 5675 50  0001 C CNN
+F 1 "PWR_FLAG" H 3200 5774 50  0000 C CNN
+F 2 "" H 3200 5600 50  0001 C CNN
+F 3 "~" H 3200 5600 50  0001 C CNN
+	1    3200 5600
+	1    0    0    -1
+$EndComp
+$Comp
+L power:PWR_FLAG #FLG0106
+U 1 1 5C6537D3
+P 2750 5600
+F 0 "#FLG0106" H 2750 5675 50  0001 C CNN
+F 1 "PWR_FLAG" H 2750 5774 50  0000 C CNN
+F 2 "" H 2750 5600 50  0001 C CNN
+F 3 "~" H 2750 5600 50  0001 C CNN
+	1    2750 5600
+	1    0    0    -1
+$EndComp
+$Comp
+L power:GNDA #PWR0132
+U 1 1 5C650B28
+P 3200 5600
+F 0 "#PWR0132" H 3200 5350 50  0001 C CNN
+F 1 "GNDA" H 3205 5427 50  0000 C CNN
+F 2 "" H 3200 5600 50  0001 C CNN
+F 3 "" H 3200 5600 50  0001 C CNN
+	1    3200 5600
+	1    0    0    -1
+$EndComp
+$Comp
+L power:GNDD #PWR0131
+U 1 1 5C650A70
+P 2750 5600
+F 0 "#PWR0131" H 2750 5350 50  0001 C CNN
+F 1 "GNDD" H 2754 5445 50  0000 C CNN
+F 2 "" H 2750 5600 50  0001 C CNN
+F 3 "" H 2750 5600 50  0001 C CNN
+	1    2750 5600
+	1    0    0    -1
+$EndComp
+Wire Wire Line
+	850  2700 900  2700
+Wire Wire Line
+	850  3950 900  3950
+$Comp
+L power:PWR_FLAG #FLG0101
+U 1 1 5C6648F6
+P 2750 6100
+F 0 "#FLG0101" H 2750 6175 50  0001 C CNN
+F 1 "PWR_FLAG" H 2750 6274 50  0000 C CNN
+F 2 "" H 2750 6100 50  0001 C CNN
+F 3 "~" H 2750 6100 50  0001 C CNN
+	1    2750 6100
+	1    0    0    -1
+$EndComp
+$Comp
+L power:+5V #PWR0114
+U 1 1 5C6655B8
+P 2750 6100
+F 0 "#PWR0114" H 2750 5950 50  0001 C CNN
+F 1 "+5V" H 2765 6273 50  0000 C CNN
+F 2 "" H 2750 6100 50  0001 C CNN
+F 3 "" H 2750 6100 50  0001 C CNN
+	1    2750 6100
+	-1   0    0    1
+$EndComp
 $EndSCHEMATC

Commit message: Misc changes
Parts:
- added C26, C27: 4.7u, Capacitor_SMD:C_0603_1608Metric_Pad1.05x0.95mm_HandSolder, symbol Device:C
- added C?: C, symbol Device:C
- added D1: B5817WS-SJ, Diode_SMD:D_SOD-323_HandSoldering, symbol Device:D_Schottky
- added L3: 4.7u, Inductor_SMD:L_Taiyo-Yuden_NR-40xx_HandSoldering, symbol Device:L_Core_Ferrite
- added R17: 820k, Resistor_SMD:R_0603_1608Metric_Pad1.05x0.95mm_HandSolder, symbol Device:R
- added R18: 18k, Resistor_SMD:R_0603_1608Metric_Pad1.05x0.95mm_HandSolder, symbol Device:R
- added U9: MT3608, Package_TO_SOT_SMD:SOT-23-6, symbol Regulator_Switching:LM27313XMF
- added U?: TPS54336ADDA, Package_SO:TI_SO-PowerPAD-8_ThermalVias, symbol Regulator_Switching:TPS54336ADDA
- L1, L2: footprint Inductor_SMD:L_Bourns-SRN4018 -> Inductor_SMD:L_Taiyo-Yuden_NR-40xx_HandSoldering
Connections:
- net +24V: now also C26.1, C?.1, L3.2, U9.4 (EN), U9.5 (VIN), U?.2 (VIN)
- net GND: now also C26.2, C27.2, C?.2, R18.2, U9.2 (GND)
- new net: D1.2 (A), L3.1, U9.1 (SW)
- new net: R17.2, R18.1, U9.3 (FB)
- new net +28V: C27.1, D1.1 (K), R17.1
Other:
- note added: ".6/28=(18kohm/(18kohm+820kohm))\nActually 27.93V"
Changed lines of the file:
@@
 EESchema Schematic File Version 4
 LIBS:solder-station-cache
-EELAYER 26 0
+EELAYER 29 0
 EELAYER END
 $Descr A4 11693 8268
@@
 F 0 "L1" V 2222 1250 50  0000 C CNN
 F 1 "4.7u" V 2313 1250 50  0000 C CNN
-F 2 "Inductor_SMD:L_Bourns-SRN4018" H 2400 1250 50  0001 C CNN
+F 2 "Inductor_SMD:L_Taiyo-Yuden_NR-40xx_HandSoldering" H 2400 1250 50  0001 C CNN
 F 3 "~" H 2400 1250 50  0001 C CNN
 	1    2400 1250
@@
 F 0 "L2" V 3722 1250 50  0000 C CNN
 F 1 "4.7u" V 3813 1250 50  0000 C CNN
-F 2 "Inductor_SMD:L_Bourns-SRN4018" H 3900 1250 50  0001 C CNN
+F 2 "Inductor_SMD:L_Taiyo-Yuden_NR-40xx_HandSoldering" H 3900 1250 50  0001 C CNN
 F 3 "~" H 3900 1250 50  0001 C CNN
 	1    3900 1250
@@
 	-1   0    0    1
 $EndComp
+$Comp
+L Regulator_Switching:LM27313XMF U9
+U 1 1 5C65F2D6
+P 7450 1450
+F 0 "U9" H 7450 1817 50  0000 C CNN
+F 1 "MT3608" H 7450 1726 50  0000 C CNN
+F 2 "Package_TO_SOT_SMD:SOT-23-6" H 7500 1200 50  0001 L CIN
+F 3 "https://datasheet.lcsc.com/szlcsc/XI-AN-Aerosemi-Tech-MT3608_C84817.pdf" H 7450 1550 50  0001 C CNN
+	1    7450 1450
+	1    0    0    -1
+$EndComp
+$Comp
+L Device:C C26
+U 1 1 5C65F564
+P 6850 1500
+F 0 "C26" H 6965 1546 50  0000 L CNN
+F 1 "4.7u" H 6965 1455 50  0000 L CNN
+F 2 "Capacitor_SMD:C_0603_1608Metric_Pad1.05x0.95mm_HandSolder" H 6888 1350 50  0001 C CNN
+F 3 "~" H 6850 1500 50  0001 C CNN
+	1    6850 1500
+	1    0    0    -1
+$EndComp
+$Comp
+L power:+24V #PWR0115
+U 1 1 5C65F56C
+P 6700 1350
+F 0 "#PWR0115" H 6700 1200 50  0001 C CNN
+F 1 "+24V" V 6715 1478 50  0000 L CNN
+F 2 "" H 6700 1350 50  0001 C CNN
+F 3 "" H 6700 1350 50  0001 C CNN
+	1    6700 1350
+	0    -1   -1   0
+$EndComp
+$Comp
+L power:GND #PWR0123
+U 1 1 5C65F575
+P 7450 1750
+F 0 "#PWR0123" H 7450 1500 50  0001 C CNN
+F 1 "GND" H 7455 1577 50  0000 C CNN
+F 2 "" H 7450 1750 50  0001 C CNN
+F 3 "" H 7450 1750 50  0001 C CNN
+	1    7450 1750
+	1    0    0    -1
+$EndComp
+Wire Wire Line
+	7150 1350 7150 1550
+Connection ~ 7150 1350
+Wire Wire Line
+	6850 1750 6850 1650
+Wire Wire Line
+	6850 1350 7150 1350
+Wire Wire Line
+	6700 1350 6850 1350
+Connection ~ 6850 1350
+$Comp
+L Device:L_Core_Ferrite L3
+U 1 1 5C66C052
+P 7450 900
+F 0 "L3" V 7272 900 50  0000 C CNN
+F 1 "4.7u" V 7363 900 50  0000 C CNN
+F 2 "Inductor_SMD:L_Taiyo-Yuden_NR-40xx_HandSoldering" H 7450 900 50  0001 C CNN
+F 3 "~" H 7450 900 50  0001 C CNN
+F 4 "1.5A" V 7450 900 50  0001 C CNN "Max current"
+	1    7450 900
+	0    1    1    0
+$EndComp
+Wire Wire Line
+	7150 1350 7150 900
+Wire Wire Line
+	7150 900  7300 900
+Wire Wire Line
+	7600 900  7750 900
+Wire Wire Line
+	7750 900  7750 1350
+$Comp
+L Device:R R18
+U 1 1 5C66E8D3
+P 8050 1600
+F 0 "R18" H 8120 1646 50  0000 L CNN
+F 1 "18k" H 8120 1555 50  0000 L CNN
+F 2 "Resistor_SMD:R_0603_1608Metric_Pad1.05x0.95mm_HandSolder" V 7980 1600 50  0001 C CNN
+F 3 "~" H 8050 1600 50  0001 C CNN
+	1    8050 1600
+	1    0    0    -1
+$EndComp
+$Comp
+L Device:R R17
+U 1 1 5C66E986
+P 8050 1300
+F 0 "R17" H 8120 1346 50  0000 L CNN
+F 1 "820k" H 8120 1255 50  0000 L CNN
+F 2 "Resistor_SMD:R_0603_1608Metric_Pad1.05x0.95mm_HandSolder" V 7980 1300 50  0001 C CNN
+F 3 "~" H 8050 1300 50  0001 C CNN
+	1    8050 1300
+	1    0    0    -1
+$EndComp
+$Comp
+L Device:D_Schottky D1
+U 1 1 5C66FB5F
+P 7900 900
+F 0 "D1" H 7900 684 50  0000 C CNN
+F 1 "B5817WS-SJ" H 7900 775 50  0000 C CNN
+F 2 "Diode_SMD:D_SOD-323_HandSoldering" H 7900 900 50  0001 C CNN
+F 3 "https://datasheet.lcsc.com/szlcsc/MDD-Jiangsu-Yutai-Elec-B5817WS-SJ_C114023.pdf" H 7900 900 50  0001 C CNN
+	1    7900 900
+	-1   0    0    1
+$EndComp
+Connection ~ 7750 900
+Wire Wire Line
+	7450 1750 8050 1750
+Connection ~ 7450 1750
+Wire Wire Line
+	8050 1150 8050 900
+Wire Wire Line
+	7750 1550 7900 1550
+Wire Wire Line
+	7900 1550 7900 1450
+Wire Wire Line
+	7900 1450 8050 1450
+Connection ~ 8050 1450
+$Comp
+L Device:C C27
+U 1 1 5C6786AD
+P 8400 1500
+F 0 "C27" H 8515 1546 50  0000 L CNN
+F 1 "4.7u" H 8515 1455 50  0000 L CNN
+F 2 "Capacitor_SMD:C_0603_1608Metric_Pad1.05x0.95mm_HandSolder" H 8438 1350 50  0001 C CNN
+F 3 "~" H 8400 1500 50  0001 C CNN
+	1    8400 1500
+	1    0    0    -1
+$EndComp
+Wire Wire Line
+	8400 1350 8400 900
+Wire Wire Line
+	8400 900  8050 900
+Connection ~ 8050 900
+Wire Wire Line
+	8050 1750 8400 1750
+Wire Wire Line
+	8400 1750 8400 1650
+Connection ~ 8050 1750
+Wire Wire Line
+	6850 1750 7450 1750
+$Comp
+L power:+28V #PWR0133
+U 1 1 5C67CEE0
+P 8600 1350
+F 0 "#PWR0133" H 8600 1200 50  0001 C CNN
+F 1 "+28V" V 8615 1478 50  0000 L CNN
+F 2 "" H 8850 1400 50  0001 C CNN
+F 3 "" H 8850 1400 50  0001 C CNN
+	1    8600 1350
+	0    1    1    0
+$EndComp
+Text Notes 7600 1950 0    50   ~ 0
+.6/28=(18kohm/(18kohm+820kohm))\nActually 27.93V
+Wire Wire Line
+	8600 1350 8400 1350
+Connection ~ 8400 1350
+$Comp
+L Regulator_Switching:TPS54336ADDA U?
+U 1 1 5CC853B8
+P 5000 3350
+F 0 "U?" H 5000 3817 50  0000 C CNN
+F 1 "TPS54336ADDA" H 5000 3726 50  0000 C CNN
+F 2 "Package_SO:TI_SO-PowerPAD-8_ThermalVias" H 5900 3000 50  0001 C CNN
+F 3 "http://www.ti.com/lit/ds/symlink/tps54336a.pdf" H 6000 2900 50  0001 C CNN
+	1    5000 3350
+	1    0    0    -1
+$EndComp
+$Comp
+L power:+24V #PWR?
+U 1 1 5CC8CA7B
+P 3950 3000
+F 0 "#PWR?" H 3950 2850 50  0001 C CNN
+F 1 "+24V" H 3965 3173 50  0000 C CNN
+F 2 "" H 3950 3000 50  0001 C CNN
+F 3 "" H 3950 3000 50  0001 C CNN
+	1    3950 3000
+	1    0    0    -1
+$EndComp
+$Comp
+L Device:C C?
+U 1 1 5CC90A62
+P 3950 3300
+F 0 "C?" H 4065 3346 50  0000 L CNN
+F 1 "C" H 4065 3255 50  0000 L CNN
+F 2 "" H 3988 3150 50  0001 C CNN
+F 3 "~" H 3950 3300 50  0001 C CNN
+	1    3950 3300
+	1    0    0    -1
+$EndComp
+Wire Wire Line
+	4500 3150 3950 3150
+Wire Wire Line
+	3950 3150 3950 3000
+Connection ~ 3950 3150
+$Comp
+L power:GND #PWR?
+U 1 1 5CC97E7D
+P 3950 3450
+F 0 "#PWR?" H 3950 3200 50  0001 C CNN
+F 1 "GND" H 3955 3277 50  0000 C CNN
+F 2 "" H 3950 3450 50  0001 C CNN
+F 3 "" H 3950 3450 50  0001 C CNN
+	1    3950 3450
+	1    0    0    -1
+$EndComp
 $EndSCHEMATC
