File: solder-station.sch (KiCad schematic (older format))
At the start: 43 parts, among them J1 Temp Sensor, J2 Heating Element, J3 SWD ISP, J4 STM_UART, Q1 BC856BDW1, Q2 NTMFS4937N, Q3 L2N7002M3T5G, Q4 L2N7002M3T5G, U1 LM75B, U2 74LVC1G58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

Commit message: Fix bug where mosfet would not work & reduce cm^2
Parts:
- removed Q1: BC856BDW1, Package_TO_SOT_SMD:SOT-363_SC-70-6_Handsoldering, symbol Transistor_BJT:BC856BDW1
- removed Q2: NTMFS4937N, solder-station:ON_S-SO-8_5.3x6.2mm_P1.27mm_TAB488AA, symbol solder-station:NTMFS4937N
- removed U2: 74LVC1G58, Package_TO_SOT_SMD:SOT-363_SC-70-6_Handsoldering, symbol 74xGxx:74LVC1G58
- added Q1, Q2: MBT3946DW1T1, Package_TO_SOT_SMD:SOT-363_SC-70-6, symbol Transistor_BJT:MBT3946DW1T1
- added Q5: FDMS6681Z, Package_TO_SOT_SMD:LFPAK56_ThermalVias-1, symbol solder-station:FDMS6681Z
- added R10: 10k, Resistor_SMD:R_0603_1608Metric_Pad1.05x0.95mm_HandSolder, symbol Device:R
- added R11: 0, Resistor_SMD:R_0603_1608Metric_Pad1.05x0.95mm_HandSolder, symbol Device:R
- added U2: 74LVC1G57, Package_TO_SOT_SMD:SOT-363_SC-70-6, symbol 74xGxx:74LVC1G57
- F1: value 20A -> 10A
Connections:
- net labels added: VCC
- net labels removed: +10V
- wire segments 85 -> 93
Other:
- note added: "S P | O\n0 0 | 1\n0 1 | 0\n1 0 | 1\n1 1 | 1"
- note removed: "S P | O\n0 0 | 0\n0 1 | 1\n1 0 | 0\n1 1 | 1"
- moved on the sheet: C1, C10, C11, C12, C13, C14, C15, C16, C2, C4, C5, C6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

Commit message: Add beginnings of a PSU & power filtering
Parts:
- R3: value DNP -> 3.3
Changed lines of the file:
@@
 $Descr A4 11693 8268
 encoding utf-8
-Sheet 1 1
+Sheet 1 2
 Title ""
 Date ""
@@
 P 4550 1650
 F 0 "R3" H 4620 1696 50  0000 L CNN
-F 1 "DNP" H 4620 1605 50  0000 L CNN
+F 1 "3.3" H 4620 1605 50  0000 L CNN
 F 2 "Resistor_SMD:R_0603_1608Metric_Pad1.05x0.95mm_HandSolder" V 4480 1650 50  0001 C CNN
 F 3 "~" H 4550 1650 50  0001 C CNN
@@
 	1    0    0    -1
 $EndComp
+$Sheet
+S 3050 6200 2250 1050
+U 5C542287
+F0 "Power supply" 50
+F1 "power.sch" 50
+$EndSheet
 $EndSCHEMATC

Commit message: Add power supplies
Parts:
- U2: symbol 74xGxx:74LVC1G57 -> solder-station:74LVC1G57
Connections:
- net labels added: GNDD
- net labels removed: GNDPWR, VCC
- wire segments 93 -> 99
Other:
- moved on the sheet: C1, C2, F1, Q1A, Q1B, Q2A, Q5, R10, R11

Commit message: Move some things around
Parts:
- J1: footprint TerminalBlock:TerminalBlock_Altech_AK300-2_P5.00mm -> Connector_PinHeader_1.27mm:PinHeader_1x02_P1.27mm_Vertical
- J2: footprint TerminalBlock:TerminalBlock_Altech_AK300-2_P5.00mm -> TerminalBlock_MetzConnect:TerminalBlock_MetzConnect_Type011_RT05502HBWC_1x02_P5.00mm_Horizontal
- J3: value SWD ISP -> ISP
- J4: value STM_UART -> I2C
Connections:
- net +3V3: now also J4.1 (Pin_1); no longer J4.4 (Pin_4)
- net GNDA: now also U5.10 (PA4)
- net GNDD: now also C16.2, J4.2 (Pin_2), U5.1 (BOOT0), U5.11 (PA5), U5.14 (PB1); no longer J4.3 (Pin_3)
- net I2C1_SCL: now also J4.3 (Pin_3)
- net I2C1_SDA: now also J4.4 (Pin_4)
- removed net USART6_RX: J4.1 (Pin_1), U5.11 (PA5)
- removed net USART6_TX: J4.2 (Pin_2), U5.10 (PA4)
- no-connect marks 7 -> 6
Other:
- note added: "MCU I2C Interface"
- note removed: "MCU Serial Interface"
Changed lines of the file:
@@
 $Descr A4 11693 8268
 encoding utf-8
-Sheet 1 2
+Sheet 1 3
 Title ""
 Date ""
@@
 Wire Wire Line
 	8100 2450 8100 2250
-NoConn ~ 9350 2250
 Text HLabel 10350 2350 2    50   BiDi ~ 0
 I_SWDIO
@@
 P 8700 3700
 F 0 "J3" H 8779 3742 50  0000 L CNN
-F 1 "SWD ISP" H 8779 3651 50  0000 L CNN
+F 1 "ISP" H 8779 3651 50  0000 L CNN
 F 2 "Connector_PinHeader_1.27mm:PinHeader_1x05_P1.27mm_Vertical" H 8700 3700 50  0001 C CNN
 F 3 "~" H 8700 3700 50  0001 C CNN
@@
 	1    0    0    -1
 $EndComp
-Wire Wire Line
-	9000 2150 9350 2150
 Text HLabel 10350 2150 2    50   BiDi ~ 0
 I2C1_SCL
@@
 F 0 "J2" H 5180 1546 50  0000 L CNN
 F 1 "Heating Element" H 5180 1501 50  0001 L CNN
-F 2 "TerminalBlock:TerminalBlock_Altech_AK300-2_P5.00mm" H 5100 1600 50  0001 C CNN
+F 2 "TerminalBlock_MetzConnect:TerminalBlock_MetzConnect_Type011_RT05502HBWC_1x02_P5.00mm_Horizontal" H 5100 1600 50  0001 C CNN
 F 3 "~" H 5100 1600 50  0001 C CNN
 	1    5100 1600
@@
 F 0 "J1" H 3920 3917 50  0000 C CNN
 F 1 "Temp Sensor" H 4080 4051 50  0001 L CNN
-F 2 "TerminalBlock:TerminalBlock_Altech_AK300-2_P5.00mm" H 4000 4150 50  0001 C CNN
+F 2 "Connector_PinHeader_1.27mm:PinHeader_1x02_P1.27mm_Vertical" H 4000 4150 50  0001 C CNN
 F 3 "~" H 4000 4150 50  0001 C CNN
 	1    4000 4150
@@
 	4600 1100 4900 1100
 Connection ~ 6850 800
-NoConn ~ 9350 2450
 Wire Notes Line
 	7950 550  10900 550
@@
 	1    0    0    -1
 $EndComp
-Text HLabel 10350 1750 2    50   Output ~ 0
-USART6_TX
-Text HLabel 10350 1850 2    50   Input ~ 0
-USART6_RX
-$Comp
-L power:+3.3V #PWR027
-U 1 1 5C6FF887
-P 9900 3500
-F 0 "#PWR027" H 9900 3350 50  0001 C CNN
-F 1 "+3.3V" V 9915 3628 50  0000 L CNN
-F 2 "" H 9900 3500 50  0001 C CNN
-F 3 "" H 9900 3500 50  0001 C CNN
-	1    9900 3500
-	0    -1   -1   0
-$EndComp
-Text HLabel 9900 3700 0    50   Input ~ 0
-USART6_TX
-Text HLabel 9900 3800 0    50   Output ~ 0
-USART6_RX
 Wire Notes Line
 	9350 3300 10650 3300
@@
 	10650 3300 10650 4200
 Text Notes 9400 4150 0    50   ~ 0
-MCU Serial Interface
+MCU I2C Interface
 Wire Notes Line
 	9350 3300 9350 4200
@@
 L Connector:Conn_01x04_Male J4
 U 1 1 5C70758E
-P 10100 3700
-F 0 "J4" H 10073 3580 50  0000 R CNN
-F 1 "STM_UART" H 10073 3671 50  0000 R CNN
-F 2 "Connector_PinHeader_1.27mm:PinHeader_1x04_P1.27mm_Vertical" H 10100 3700 50  0001 C CNN
-F 3 "~" H 10100 3700 50  0001 C CNN
-	1    10100 3700
-	-1   0    0    1
+P 10100 3600
+F 0 "J4" H 10073 3480 50  0000 R CNN
+F 1 "I2C" H 10073 3571 50  0000 R CNN
+F 2 "Connector_PinHeader_1.27mm:PinHeader_1x04_P1.27mm_Vertical" H 10100 3600 50  0001 C CNN
+F 3 "~" H 10100 3600 50  0001 C CNN
+	1    10100 3600
+	-1   0    0    -1
 $EndComp
 $Comp
@@
 $EndComp
 $Comp
+L power:GNDD #PWR0113
+U 1 1 5C5FC6D0
+P 8500 3600
+F 0 "#PWR0113" H 8500 3350 50  0001 C CNN
+F 1 "GNDD" V 8504 3490 50  0000 R CNN
+F 2 "" H 8500 3600 50  0001 C CNN
+F 3 "" H 8500 3600 50  0001 C CNN
+	1    8500 3600
+	0    1    1    0
+$EndComp
+$Comp
+L Device:C_Small C3
+U 1 1 5C5FD0ED
+P 800 3750
+F 0 "C3" H 892 3796 50  0000 L CNN
+F 1 "1u" H 892 3705 50  0000 L CNN
+F 2 "Capacitor_SMD:C_0603_1608Metric_Pad1.05x0.95mm_HandSolder" H 800 3750 50  0001 C CNN
+F 3 "~" H 800 3750 50  0001 C CNN
+	1    800  3750
+	1    0    0    -1
+$EndComp
+Wire Wire Line
+	800  3650 1200 3650
+Connection ~ 1200 3650
+Wire Wire Line
+	1200 3650 1200 3750
+Wire Wire Line
+	800  3850 800  4150
+Connection ~ 800  4150
+$Comp
+L power:GNDD #PWR0107
+U 1 1 5C614115
+P 1950 1800
+F 0 "#PWR0107" H 1950 1550 50  0001 C CNN
+F 1 "GNDD" H 1954 1645 50  0000 C CNN
+F 2 "" H 1950 1800 50  0001 C CNN
+F 3 "" H 1950 1800 50  0001 C CNN
+	1    1950 1800
+	1    0    0    -1
+$EndComp
+$Comp
+L power:GND #PWR0121
+U 1 1 5C614A41
+P 2550 1800
+F 0 "#PWR0121" H 2550 1550 50  0001 C CNN
+F 1 "GND" H 2555 1627 50  0000 C CNN
+F 2 "" H 2550 1800 50  0001 C CNN
+F 3 "" H 2550 1800 50  0001 C CNN
+	1    2550 1800
+	1    0    0    -1
+$EndComp
+$Comp
+L power:GNDD #PWR0122
+U 1 1 5C615228
+P 1150 1800
+F 0 "#PWR0122" H 1150 1550 50  0001 C CNN
+F 1 "GNDD" V 1154 1690 50  0000 R CNN
+F 2 "" H 1150 1800 50  0001 C CNN
+F 3 "" H 1150 1800 50  0001 C CNN
+	1    1150 1800
+	0    1    1    0
+$EndComp
+$Comp
+L power:GNDD #PWR0125
+U 1 1 5C635D5D
+P 1450 2200
+F 0 "#PWR0125" H 1450 1950 50  0001 C CNN
+F 1 "GNDD" H 1454 2045 50  0000 C CNN
+F 2 "" H 1450 2200 50  0001 C CNN
+F 3 "" H 1450 2200 50  0001 C CNN
+	1    1450 2200
+	1    0    0    -1
+$EndComp
+$Comp
+L power:+3.3V #PWR0126
+U 1 1 5C63D96A
+P 1450 1600
+F 0 "#PWR0126" H 1450 1450 50  0001 C CNN
+F 1 "+3.3V" H 1465 1773 50  0000 C CNN
+F 2 "" H 1450 1600 50  0001 C CNN
+F 3 "" H 1450 1600 50  0001 C CNN
+	1    1450 1600
+	1    0    0    -1
+$EndComp
+Wire Wire Line
+	1400 1000 1950 1000
+Connection ~ 1950 1000
+Wire Notes Line
+	550  550  550  2550
+Wire Notes Line
+	550  2550 3800 2550
+Wire Notes Line
+	3800 550  3800 2550
+Wire Notes Line
+	550  2400 3800 2400
+Wire Wire Line
+	9000 2150 9350 2150
+Wire Wire Line
+	9350 2450 9350 2650
+Wire Wire Line
+	9350 2650 9850 2650
+Connection ~ 9850 2650
+$Comp
+L power:GNDD #PWR0127
+U 1 1 5C5B6191
+P 9100 1550
+F 0 "#PWR0127" H 9100 1300 50  0001 C CNN
+F 1 "GNDD" H 9104 1395 50  0000 C CNN
+F 2 "" H 9100 1550 50  0001 C CNN
+F 3 "" H 9100 1550 50  0001 C CNN
+	1    9100 1550
+	1    0    0    -1
+$EndComp
+NoConn ~ 9350 2250
+$Comp
+L power:GNDA #PWR0128
+U 1 1 5C5B008A
+P 10350 1750
+F 0 "#PWR0128" H 10350 1500 50  0001 C CNN
+F 1 "GNDA" V 10355 1622 50  0000 R CNN
+F 2 "" H 10350 1750 50  0001 C CNN
+F 3 "" H 10350 1750 50  0001 C CNN
+	1    10350 1750
+	0    -1   -1   0
+$EndComp
+$Comp
+L power:GNDD #PWR0129
+U 1 1 5C5B3D65
+P 10350 1850
+F 0 "#PWR0129" H 10350 1600 50  0001 C CNN
+F 1 "GNDD" V 10354 1740 50  0000 R CNN
+F 2 "" H 10350 1850 50  0001 C CNN
+F 3 "" H 10350 1850 50  0001 C CNN
+	1    10350 1850
+	0    -1   -1   0
+$EndComp
+Text HLabel 9900 3700 0    50   BiDi ~ 0
+I2C1_SCL
+Text HLabel 9900 3800 0    50   BiDi ~ 0
+I2C1_SDA
+$Comp
 L power:GNDD #PWR0112
 U 1 1 5C5FC4D9
@@
 $EndComp
 $Comp
-L power:GNDD #PWR0113
-U 1 1 5C5FC6D0
-P 8500 3600
-F 0 "#PWR0113" H 8500 3350 50  0001 C CNN
-F 1 "GNDD" V 8504 3490 50  0000 R CNN
-F 2 "" H 8500 3600 50  0001 C CNN
-F 3 "" H 8500 3600 50  0001 C CNN
-	1    8500 3600
-	0    1    1    0
-$EndComp
-$Comp
-L Device:C_Small C3
-U 1 1 5C5FD0ED
-P 800 3750
-F 0 "C3" H 892 3796 50  0000 L CNN
-F 1 "1u" H 892 3705 50  0000 L CNN
-F 2 "Capacitor_SMD:C_0603_1608Metric_Pad1.05x0.95mm_HandSolder" H 800 3750 50  0001 C CNN
-F 3 "~" H 800 3750 50  0001 C CNN
-	1    800  3750
-	1    0    0    -1
-$EndComp
-Wire Wire Line
-	800  3650 1200 3650
-Connection ~ 1200 3650
-Wire Wire Line
-	1200 3650 1200 3750
-Wire Wire Line
-	800  3850 800  4150
-Connection ~ 800  4150
-$Comp
-L power:GNDD #PWR0107
-U 1 1 5C614115
-P 1950 1800
-F 0 "#PWR0107" H 1950 1550 50  0001 C CNN
-F 1 "GNDD" H 1954 1645 50  0000 C CNN
-F 2 "" H 1950 1800 50  0001 C CNN
-F 3 "" H 1950 1800 50  0001 C CNN
-	1    1950 1800
-	1    0    0    -1
-$EndComp
-$Comp
-L power:GND #PWR0121
-U 1 1 5C614A41
-P 2550 1800
-F 0 "#PWR0121" H 2550 1550 50  0001 C CNN
-F 1 "GND" H 2555 1627 50  0000 C CNN
-F 2 "" H 2550 1800 50  0001 C CNN
-F 3 "" H 2550 1800 50  0001 C CNN
-	1    2550 1800
-	1    0    0    -1
-$EndComp
-$Comp
-L power:GNDD #PWR0122
-U 1 1 5C615228
-P 1150 1800
-F 0 "#PWR0122" H 1150 1550 50  0001 C CNN
-F 1 "GNDD" V 1154 1690 50  0000 R CNN
-F 2 "" H 1150 1800 50  0001 C CNN
-F 3 "" H 1150 1800 50  0001 C CNN
-	1    1150 1800
-	0    1    1    0
-$EndComp
-$Comp
-L power:GNDD #PWR0125
-U 1 1 5C635D5D
-P 1450 2200
-F 0 "#PWR0125" H 1450 1950 50  0001 C CNN
-F 1 "GNDD" H 1454 2045 50  0000 C CNN
-F 2 "" H 1450 2200 50  0001 C CNN
-F 3 "" H 1450 2200 50  0001 C CNN
-	1    1450 2200
-	1    0    0    -1
-$EndComp
-$Comp
-L power:+3.3V #PWR0126
-U 1 1 5C63D96A
-P 1450 1600
-F 0 "#PWR0126" H 1450 1450 50  0001 C CNN
-F 1 "+3.3V" H 1465 1773 50  0000 C CNN
-F 2 "" H 1450 1600 50  0001 C CNN
-F 3 "" H 1450 1600 50  0001 C CNN
-	1    1450 1600
-	1    0    0    -1
-$EndComp
-Wire Wire Line
-	1400 1000 1950 1000
-Connection ~ 1950 1000
-Wire Notes Line
-	550  550  550  2550
-Wire Notes Line
-	550  2550 3800 2550
-Wire Notes Line
-	3800 550  3800 2550
-Wire Notes Line
-	550  2400 3800 2400
+L power:+3.3V #PWR027
+U 1 1 5C6FF887
+P 9900 3500
+F 0 "#PWR027" H 9900 3350 50  0001 C CNN
+F 1 "+3.3V" V 9915 3628 50  0000 L CNN
+F 2 "" H 9900 3500 50  0001 C CNN
+F 3 "" H 9900 3500 50  0001 C CNN
+	1    9900 3500
+	0    -1   -1   0
+$EndComp
 $EndSCHEMATC

Commit message: Add test points
Parts:
- added TP1: A_THERMO, symbol Connector:TestPoint
- added TP2: A_IRON, symbol Connector:TestPoint
- C14, C7, C8: value 10n -> .1u
- C4, C6: value 1n -> .1u
- C5: value 10n -> 1u
- J4: symbol Connector:Conn_01x04_Male -> Connector_Generic:Conn_01x04
Connections:
- net A_IRON: now also TP2.1
- net A_THERMO: now also TP1.1
Changed lines of the file:
@@
 $Descr A4 11693 8268
 encoding utf-8
-Sheet 1 3
+Sheet 1 2
 Title ""
 Date ""
@@
 P 10100 950
 F 0 "C14" H 10192 996 50  0000 L CNN
-F 1 "10n" H 10192 905 50  0000 L CNN
+F 1 ".1u" H 10192 905 50  0000 L CNN
 F 2 "Capacitor_SMD:C_0603_1608Metric_Pad1.05x0.95mm_HandSolder" H 10100 950 50  0001 C CNN
 F 3 "~" H 10100 950 50  0001 C CNN
@@
 	4450 1800 4450 1650
 NoConn ~ 4300 1800
-Text HLabel 7250 1450 2    50   Output ~ 0
+Text HLabel 7300 1450 2    50   Output ~ 0
 A_IRON
 Wire Notes Line
@@
 P 6950 900
 F 0 "C8" H 7042 946 50  0000 L CNN
-F 1 "10n" H 7042 855 50  0000 L CNN
+F 1 ".1u" H 7042 855 50  0000 L CNN
 F 2 "Capacitor_SMD:C_0603_1608Metric_Pad1.05x0.95mm_HandSolder" H 6950 900 50  0001 C CNN
 F 3 "~" H 6950 900 50  0001 C CNN
@@
 P 4850 4100
 F 0 "C5" H 4942 4146 50  0000 L CNN
-F 1 "10n" H 4942 4055 50  0000 L CNN
+F 1 "1u" H 4942 4055 50  0000 L CNN
 F 2 "Capacitor_SMD:C_0603_1608Metric_Pad1.05x0.95mm_HandSolder" H 4850 4100 50  0001 C CNN
 F 3 "~" H 4850 4100 50  0001 C CNN
@@
 P 4850 3900
 F 0 "C4" H 4942 3946 50  0000 L CNN
-F 1 "1n" H 4942 3855 50  0000 L CNN
+F 1 ".1u" H 4942 3855 50  0000 L CNN
 F 2 "Capacitor_SMD:C_0603_1608Metric_Pad1.05x0.95mm_HandSolder" H 4850 3900 50  0001 C CNN
 F 3 "~" H 4850 3900 50  0001 C CNN
@@
 P 4850 4300
 F 0 "C6" H 4942 4346 50  0000 L CNN
-F 1 "1n" H 4942 4255 50  0000 L CNN
+F 1 ".1u" H 4942 4255 50  0000 L CNN
 F 2 "Capacitor_SMD:C_0603_1608Metric_Pad1.05x0.95mm_HandSolder" H 4850 4300 50  0001 C CNN
 F 3 "~" H 4850 4300 50  0001 C CNN
@@
 	5750 4700 5850 4700
 Wire Wire Line
-	5850 4700 5850 4100
+	5850 4700 5850 4250
 Wire Wire Line
 	5850 4100 5700 4100
@@
 P 5500 3800
 F 0 "C7" V 5271 3800 50  0000 C CNN
-F 1 "10n" V 5362 3800 50  0000 C CNN
+F 1 ".1u" V 5362 3800 50  0000 C CNN
 F 2 "Capacitor_SMD:C_0603_1608Metric_Pad1.05x0.95mm_HandSolder" H 5500 3800 50  0001 C CNN
 F 3 "~" H 5500 3800 50  0001 C CNN
@@
 	9350 3300 9350 4200
 $Comp
-L Connector:Conn_01x04_Male J4
+L Connector_Generic:Conn_01x04 J4
 U 1 1 5C70758E
 P 10100 3600
-F 0 "J4" H 10073 3480 50  0000 R CNN
-F 1 "I2C" H 10073 3571 50  0000 R CNN
+F 0 "J4" H 10250 3600 50  0000 R CNN
+F 1 "I2C" H 10300 3500 50  0000 R CNN
 F 2 "Connector_PinHeader_1.27mm:PinHeader_1x04_P1.27mm_Vertical" H 10100 3600 50  0001 C CNN
 F 3 "~" H 10100 3600 50  0001 C CNN
 	1    10100 3600
-	-1   0    0    -1
+	1    0    0    -1
 $EndComp
 $Comp
@@
 	0    -1   -1   0
 $EndComp
+Wire Wire Line
+	7250 1450 7300 1450
+Wire Wire Line
+	7250 1450 7250 1550
+Connection ~ 7250 1450
+$Comp
+L Connector:TestPoint TP2
+U 1 1 5C5DBC88
+P 7250 1550
+F 0 "TP2" H 7192 1577 50  0000 R CNN
+F 1 "A_IRON" H 7192 1668 50  0000 R CNN
+F 2 "" H 7450 1550 50  0001 C CNN
+F 3 "~" H 7450 1550 50  0001 C CNN
+	1    7250 1550
+	-1   0    0    1
+$EndComp
+$Comp
+L Connector:TestPoint TP1
+U 1 1 5C5DC495
+P 5850 4250
+F 0 "TP1" V 5804 4437 50  0000 L CNN
+F 1 "A_THERMO" V 5895 4437 50  0000 L CNN
+F 2 "" H 6050 4250 50  0001 C CNN
+F 3 "~" H 6050 4250 50  0001 C CNN
+	1    5850 4250
+	0    1    1    0
+$EndComp
+Connection ~ 5850 4250
+Wire Wire Line
+	5850 4250 5850 4100
 $EndSCHEMATC

Commit message: Fix DRC issues
Connections:
- net A_THERMO renamed A_THERM
Changed lines of the file:
@@
 	8100 1850 8700 1850
 Wire Wire Line
-	8700 2450 8100 2450
-Wire Wire Line
 	8100 2450 8100 2250
-Text HLabel 10350 2350 2    50   BiDi ~ 0
-I_SWDIO
-Text HLabel 10350 2450 2    50   Input ~ 0
-I_SWCLK
-Text HLabel 8550 1350 0    50   Input ~ 0
-I_RESET
 $Comp
 L power:+3.3V #PWR020
@@
 $EndComp
 Connection ~ 9000 850
-Text HLabel 8500 3700 0    50   BiDi ~ 0
-I_SWDIO
-Text HLabel 8500 3800 0    50   Input ~ 0
-I_SWCLK
-Text HLabel 8500 3900 0    50   Output ~ 0
-I_RESET
 $Comp
 L Connector_Generic:Conn_01x05 J3
@@
 	1    0    0    -1
 $EndComp
-Text HLabel 10350 2150 2    50   BiDi ~ 0
-I2C1_SCL
-Text HLabel 10350 2250 2    50   BiDi ~ 0
-I2C1_SDA
 $Comp
 L power:GNDA #PWR032
@@
 L power:GNDA #PWR017
 U 1 1 5C4FB4F8
-P 6950 1750
-F 0 "#PWR017" H 6950 1500 50  0001 C CNN
-F 1 "GNDA" H 6955 1577 50  0000 C CNN
-F 2 "" H 6950 1750 50  0001 C CNN
-F 3 "" H 6950 1750 50  0001 C CNN
-	1    6950 1750
-	1    0    0    -1
-$EndComp
-Wire Wire Line
-	6850 1750 6950 1750
-Connection ~ 6950 1750
+P 6850 1750
+F 0 "#PWR017" H 6850 1500 50  0001 C CNN
+F 1 "GNDA" H 6855 1577 50  0000 C CNN
+F 2 "" H 6850 1750 50  0001 C CNN
+F 3 "" H 6850 1750 50  0001 C CNN
+	1    6850 1750
+	1    0    0    -1
+$EndComp
 $Comp
 L Device:R R6
@@
 	1    0    0    -1
 $EndComp
-Text HLabel 3350 1800 2    50   Output ~ 0
-IRON_PWR
-Text HLabel 4850 1400 0    50   Input ~ 0
-IRON_PWR
 Wire Wire Line
 	4850 1400 4900 1400
@@
 Wire Wire Line
 	6300 1650 6550 1650
-Text HLabel 10350 1950 2    50   Output ~ 0
-EN_SEN
-Text HLabel 10350 2050 2    50   Output ~ 0
-EN_PWR
-Text HLabel 10350 1550 2    50   Input ~ 0
-A_IRON
 $Comp
 L Device:Q_NMOS_DGS Q3
@@
 Wire Wire Line
 	6300 1150 6300 1250
-Text HLabel 5400 2700 0    50   Input ~ 0
-EN_SEN
 Wire Wire Line
 	5400 1150 5400 1400
@@
 	4450 1800 4450 1650
 NoConn ~ 4300 1800
-Text HLabel 7300 1450 2    50   Output ~ 0
-A_IRON
 Wire Notes Line
 	7650 550  7650 3000
@@
 	-1   0    0    -1
 $EndComp
-Text HLabel 1600 4250 2    50   BiDi ~ 0
-I2C1_SCL
-Text HLabel 1600 4150 2    50   BiDi ~ 0
-I2C1_SDA
 Wire Notes Line
 	550  5050 2100 5050
@@
 Wire Wire Line
 	5100 4200 5100 4850
-Text HLabel 5950 4100 2    50   Output ~ 0
-A_THERMO
-Text HLabel 10350 1450 2    50   Input ~ 0
-A_THERMO
 Text Notes 3950 5350 0    50   ~ 0
 Filtering based on recs in analog.com/.../measuring-temp-\nusing-thermocouples\nR_fb/10kohm = (3.3V/20mV)
@@
 	1    0    0    -1
 $EndComp
-Text HLabel 1150 1900 0    50   Input ~ 0
-EN_PWR
-Text HLabel 1150 2000 0    50   Input ~ 0
-EN_SEN
 $Sheet
 S 3050 6200 2250 1050
@@
 Wire Wire Line
 	9350 2450 9350 2650
-Wire Wire Line
-	9350 2650 9850 2650
-Connection ~ 9850 2650
 $Comp
 L power:GNDD #PWR0127
@@
 	0    -1   -1   0
 $EndComp
-Text HLabel 9900 3700 0    50   BiDi ~ 0
-I2C1_SCL
-Text HLabel 9900 3800 0    50   BiDi ~ 0
-I2C1_SDA
 $Comp
 L power:GNDD #PWR0112
@@
 Wire Wire Line
 	5850 4250 5850 4100
+Text GLabel 10350 1950 2    50   Output ~ 0
+EN_SEN
+Text GLabel 10350 2050 2    50   Output ~ 0
+EN_PWR
+Text GLabel 10350 2150 2    50   BiDi ~ 0
+I2C1_SCL
+Text GLabel 10350 2250 2    50   BiDi ~ 0
+I2C1_SDA
+Text GLabel 10350 2350 2    50   BiDi ~ 0
+I_SWDIO
+Text GLabel 10350 2450 2    50   Input ~ 0
+I_SWCLK
+Text GLabel 10350 1450 2    50   Input ~ 0
+A_THERM
+Text GLabel 10350 1550 2    50   Input ~ 0
+A_IRON
+Text GLabel 8550 1350 0    50   Input ~ 0
+I_RESET
+Text GLabel 8500 3700 0    50   BiDi ~ 0
+I_SWDIO
+Text GLabel 8500 3800 0    50   Output ~ 0
+I_SWCLK
+Text GLabel 8500 3900 0    50   Output ~ 0
+I_RESET
+Text GLabel 9900 3700 0    50   BiDi ~ 0
+I2C1_SCL
+Text GLabel 9900 3800 0    50   BiDi ~ 0
+I2C1_SDA
+Text GLabel 5950 4100 2    50   Output ~ 0
+A_THERM
+Text GLabel 5400 2700 0    50   Input ~ 0
+EN_SEN
+Text GLabel 7300 1450 2    50   Output ~ 0
+A_IRON
+Text GLabel 1600 4250 2    50   BiDi ~ 0
+I2C1_SCL
+Text GLabel 1600 4150 2    50   BiDi ~ 0
+I2C1_SDA
+Text GLabel 1150 2000 0    50   Input ~ 0
+EN_SEN
+Text GLabel 1150 1900 0    50   Input ~ 0
+EN_PWR
+Text GLabel 3350 1800 2    50   Output ~ 0
+IRON_PWR
+Text GLabel 4850 1400 0    50   Input ~ 0
+IRON_PWR
+Connection ~ 8700 2450
+Wire Wire Line
+	8100 2450 8700 2450
+Connection ~ 9850 2650
+Wire Wire Line
+	9350 2650 9850 2650
+Connection ~ 6850 1750
+Wire Wire Line
+	6850 1750 6950 1750
 $EndSCHEMATC

Commit message: Misc changes
Parts:
- C10: value 4.7u -> .1u
- X1: value 20MHz -> O503220MEDH4MI; Frequency (none) -> 20M
Changed lines of the file:
@@
 EESchema Schematic File Version 4
 LIBS:solder-station-cache
-EELAYER 26 0
+EELAYER 29 0
 EELAYER END
 $Descr A4 11693 8268
@@
 P 8700 2150
 F 0 "X1" H 8800 1800 50  0000 L CNN
-F 1 "20MHz" H 8800 1900 50  0000 L CNN
+F 1 "O503220MEDH4MI" H 8800 1900 50  0001 L CNN
 F 2 "Oscillator:Oscillator_SMD_EuroQuartz_XO53-4Pin_5.0x3.2mm_HandSoldering" H 9400 1800 50  0001 C CNN
 F 3 "https://datasheet.lcsc.com/szlcsc/Yangxing-Tech-O705016MEDH4MI_C79413.pdf" H 8600 2150 50  0001 C CNN
+F 4 "20M" H 8850 1900 50  0000 C CNN "Frequency"
 	1    8700 2150
 	1    0    0    -1
@@
 P 8100 2150
 F 0 "C10" H 8192 2196 50  0000 L CNN
-F 1 "4.7u" H 8192 2105 50  0000 L CNN
+F 1 ".1u" H 8192 2105 50  0000 L CNN
 F 2 "Capacitor_SMD:C_0603_1608Metric_Pad1.05x0.95mm_HandSolder" H 8100 2150 50  0001 C CNN
 F 3 "~" H 8100 2150 50  0001 C CNN
@@
 Wire Notes Line
 	550  2400 3800 2400
-Wire Wire Line
-	9000 2150 9350 2150
 Wire Wire Line
 	9350 2450 9350 2650
@@
 Wire Wire Line
 	6850 1750 6950 1750
+Wire Wire Line
+	9000 2150 9350 2150
 $EndSCHEMATC
